File: controller_board/controller_board.kicad_pcb (KiCad board)
At the start: 2 copper layers, 38 x 90 mm, 73 parts, among them J1 USB_C_Receptacle_USB2.0, J10 input_04, J11 I2C, J12 stick, J13 input_05, J14 input_06, J15 input_07, J16 input_08, J17 I2C, J18 USB_C_Receptacle_USB2.0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

Commit message: ordered controller. create body controller model
Parts:
- added G***: LOGO, Logo:E-PIX_05x05, F.Cu at (158.1, 129.5)
- added G***: LOGO, Logo:HRU_05x05, F.Cu at (168.9, 123.2)
- added G***: LOGO, Logo:Robomech_05x05, F.Cu at (168.9, 128.3)
- moved C18 3.13 mm to (158.4, 108.0)
- moved R16 3.13 mm to (153.9, 108.0)
Routing:
- net +3V3: track 263.2 -> 266.0 mm, vias 23 -> 24
- net /ADC5: track 71.2 -> 72.9 mm
- net GND: track 61.5 -> 63.0 mm
- net /ADC6: track 77.4 -> 78.6 mm
- net /SW_stick: track 49.7 -> 50.6 mm
Other:
- board text added: "3V3"
- board text added: "ADC1"
- board text added: "ADC10"
- board text added: "ADC2"
- board text added: "ADC3"
- board text added: "ADC4"
- board text added: "ADC5"
- board text added: "ADC6"
- board text added: "ADC7"
- board text added: "ADC8"
- board text added: "ADC9"
- board text added: "BOOT"
- board text added: "E-PIX controller"
- board text added: "EN"
- board text added: "GND"
- board text added: "Robomech Factory Humanoid Robot Unit"
- board text added: "SCL"
- board text added: "SDA"
- board text added: "SW1"
- board text added: "SW_stick"
- board text added: "VDD"
- board text added: "general purpose controller board with ESP32-S2"
- board text added: "v0 2026/01/26"
